File: Micro-Flight/_autosave-RP2350_80QFN_minimal.kicad_sch (KiCad schematic)
At the start: 54 parts, among them J1 Conn_01x04_Pin, J2 Conn_01x20, J3 Conn_01x04_Pin, J5 USB_C_Receptacle_USB2.0_14P, J6 Conn_01x04_Pin, SW1 SW_Push, SW2 SW_Push, U1 RP2350_80QFN, U2 E22-900M30S, U3 W25Q128JVS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

Commit message: REV B
Other:
- note added: "Altimeter"
Changed lines of the file:
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@@
+		)
+	)
+	(text "Altimeter\n"
+		(exclude_from_sim no)
+		(at 400.558 185.928 0)
+		(effects
+			(font
+				(size 2.54 2.54)
+			)
+			(justify left bottom)
 		)
 	)
